Commit message: remove unnecessary packages, modify urdf files and add a launch file

File: src/my_robot/urdf/my_robot.xacro (robot description, xacro)
@@ -112,4 +112,6 @@
     </collision>
   </link>
+  <link name="camera_optical">
+  </link>
   <link name="hokuyo">
     <inertial>
@@ -153,4 +155,9 @@
     <axis xyz="0 1 0" rpy="0 0 0"/>
   </joint>
+  <joint name="camera_optical_joint" type="fixed">
+    <origin xyz="0 0 0" rpy="-1.5707 0 -1.5707"/>
+    <parent link="camera"/>
+    <child link="camera_optical"/>
+  </joint>
   <joint type="fixed" name="hokuyo_joint">
     <origin xyz="0.25 0 0.1" rpy="0 0 0"/>
